Commit message: cleanup URDF file

File: src/rrbot_simulation_files/rrbot_description/urdf/rrbot_description.urdf.xacro (robot description, xacro)
@@ -41,15 +41,14 @@
     </link>
     <!-- Link1 (revolute joint) -->
-    <!-- negative rotation axis to account for Gazebo rotating clockwise rather than counter-clockwise -->
     <joint name="${prefix}joint1" type="continuous">
       <parent link="${prefix}base_link" />
       <child link="${prefix}link1" />
-      <origin xyz="0 0 ${height0 + width - axel_offset}" rpy="0 1.5708 0" />
-      <axis xyz="-1 0 0" />
+      <origin xyz="0 0 ${height0 + width - axel_offset}" rpy="0 0 0" />
+      <axis xyz="0 0 1" />
       <dynamics damping="0.7" />
     </joint>
     <link name="${prefix}link1">
       <collision>
-        <origin xyz="0 0 ${height1/2 - axel_offset}" rpy="0 0 0" />
+        <origin xyz="${height1/2 - axel_offset} 0 0" rpy="0 1.5708 0" />
         <geometry>
           <box size="${width} ${width} ${height1}" />
@@ -57,5 +56,5 @@
       </collision>
       <visual>
-        <origin xyz="0 0 ${height1/2 - axel_offset}" rpy="0 0 0" />
+        <origin xyz="${height1/2 - axel_offset} 0 0" rpy="0 1.5708 0" />
         <geometry>
           <box size="${width} ${width} ${height1}" />
@@ -64,5 +63,5 @@
       </visual>
       <inertial>
-        <origin xyz="0 0 ${height1/2 - axel_offset}" rpy="0 0 0" />
+        <origin xyz="${height1/2 - axel_offset} 0 0" rpy="0 1.5708 0" />
         <mass value="${mass}" />
         <inertia
@@ -73,15 +72,14 @@
     </link>
     <!-- Link2 (revolute joint) -->
-    <!-- negative rotation axis to account for Gazebo rotating clockwise rather than counter-clockwise -->
     <joint name="${prefix}joint2" type="continuous">
       <parent link="${prefix}link1" />
       <child link="${prefix}link2" />
-      <origin xyz="-${width} 0 ${height1 - axel_offset*2}" rpy="0 0 0" />
-      <axis xyz="-1 0 0" />
+      <origin xyz="${height1 - axel_offset*2} 0 ${width}" rpy="0 0 0" />
+      <axis xyz="0 0 1" />
       <dynamics damping="0.7" />
     </joint>
     <link name="${prefix}link2">
       <collision>
-        <origin xyz="0 0 ${height2/2 - axel_offset}" rpy="0 0 0" />
+        <origin xyz="${height2/2 - axel_offset} 0 0" rpy="0 1.5708 0" />
         <geometry>
           <box size="${width} ${width} ${height2}" />
@@ -89,5 +87,5 @@
       </collision>
       <visual>
-        <origin xyz="0 0 ${height2/2 - axel_offset}" rpy="0 0 0" />
+        <origin xyz="${height2/2 - axel_offset} 0 0" rpy="0 1.5708 0" />
         <geometry>
           <box size="${width} ${width} ${height2}" />
@@ -96,5 +94,5 @@
       </visual>
       <inertial>
-        <origin xyz="0 0 ${height2/2 - axel_offset}" rpy="0 0 0" />
+        <origin xyz="${height2/2 - axel_offset} 0 0" rpy="0 1.5708 0" />
         <mass value="${mass}" />
         <inertia
@@ -108,5 +106,5 @@
       <parent link="${prefix}link2" />
       <child link="${prefix}link3" />
-      <origin xyz="0 0 ${height2 + width - axel_offset*2}" rpy="3.1416 -1.5708 0" />
+      <origin xyz="${height2 + width - axel_offset*2} 0 0" rpy="3.1416 0 0" />
       <axis xyz="0 0 1" />
       <dynamics damping="0.7" />
